File: hardware/mainboard/mainboard-reva.kicad_pcb (KiCad board)
At the start: 4 copper layers, 88 x 48 mm, 76 parts, among them J1 USB-C, J2 BATTERY, J3 SM05B-GHS-TB / ENCODER, J4 SM03B-GHS-TB / SNOOZE, J5 Molex 54550-2472 / GDEY037T03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, J6 Molex 54550-0672 / FL21 front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, J7 SPEAKER, J8 SM02B-GHS-TB / WAKE_LED, Q2 AO3400A / WAKE, U1 ESP32-S3-WROOM-1-N8, U2 BQ24074RGTR, U3 TPS62840DLCR, U4 RV-3028-C7, U5 VEML7700, U6 MAX98357AETE+T, U7 USBLC6-2SC6

Commit message: fix(mainboard): align EPD gate and I2C pull-ups with references
Parts:
- R_GDR: value 1M 1% -> 10k 1%
- R_SCL, R_SDA: value 10k -> 4.7k
Changed lines of the file:
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@@
   (footprint "Resistor_SMD:R_0603_1608Metric" (layer "F.Cu") (at 12 20)
     (property "Reference" "R_SDA" (at 0 -1.4) (layer "F.SilkS"))
-    (property "Value" "10k" (at 0 1.4) (layer "F.Fab") hide)
+    (property "Value" "4.7k" (at 0 1.4) (layer "F.Fab") hide)
     (pad "1" smd roundrect (at -0.775 0) (size 0.9 0.95) (layers "F.Cu" "F.Paste" "F.Mask") (roundrect_rratio 0.25) (net 6 "+3V3"))
     (pad "2" smd roundrect (at 0.775 0) (size 0.9 0.95) (layers "F.Cu" "F.Paste" "F.Mask") (roundrect_rratio 0.25) (net 12 "I2C_SDA"))
@@
   (footprint "Resistor_SMD:R_0603_1608Metric" (layer "F.Cu") (at 16 20)
     (property "Reference" "R_SCL" (at 0 -1.4) (layer "F.SilkS"))
-    (property "Value" "10k" (at 0 1.4) (layer "F.Fab") hide)
+    (property "Value" "4.7k" (at 0 1.4) (layer "F.Fab") hide)
     (pad "1" smd roundrect (at -0.775 0) (size 0.9 0.95) (layers "F.Cu" "F.Paste" "F.Mask") (roundrect_rratio 0.25) (net 6 "+3V3"))
     (pad "2" smd roundrect (at 0.775 0) (size 0.9 0.95) (layers "F.Cu" "F.Paste" "F.Mask") (roundrect_rratio 0.25) (net 13 "I2C_SCL"))
@@
   (footprint "Resistor_SMD:R_0603_1608Metric" (layer "F.Cu") (at 28 39)
     (property "Reference" "R_GDR" (at 0 -1.4) (layer "F.SilkS"))
-    (property "Value" "1M 1%" (at 0 1.4) (layer "F.Fab") hide)
+    (property "Value" "10k 1%" (at 0 1.4) (layer "F.Fab") hide)
     (pad "1" smd roundrect (at -0.775 0) (size 0.9 0.95) (layers "F.Cu" "F.Paste" "F.Mask") (roundrect_rratio 0.25) (net 24 "EPD_GDR"))
     (pad "2" smd roundrect (at 0.775 0) (size 0.9 0.95) (layers "F.Cu" "F.Paste" "F.Mask") (roundrect_rratio 0.25) (net 1 "GND"))

Commit message: fix(mainboard): correct EPD MOSFET pinout and add charger input decoupling
Parts:
- added C_IN: 1uF/10V, Capacitor_SMD:C_0603_1608Metric, F.Cu at (24.5, 13.0)
Connections:
- Q_EPD pad 1: EPD_GDR -> EPD_RESE
- Q_EPD pad 2: EPD_RESE -> EPD_GDR
Routing:
- net VBUS_USB: track 94.4 -> 98.9 mm, vias 5 -> 6
- net EPD_RESE: track 30.7 -> 33.7 mm, vias 3 -> 4
- net EPD_GDR: track 60.9 -> 62.6 mm
- net GND: track 105.0 -> 105.7 mm, vias 51 -> 52
Changed lines of the file:
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@@
     (pad "2" smd roundrect (at 0.95 0) (size 1 1.45) (layers "F.Cu" "F.Paste" "F.Mask") (roundrect_rratio 0.25) (net 1 "GND"))
+  )
+  (footprint "Capacitor_SMD:C_0603_1608Metric" (layer "F.Cu") (at 24.5 13.0)
+    (property "Reference" "C_IN" (at 0 -1.4) (layer "F.SilkS"))
+    (property "Value" "1uF/10V" (at 0 1.4) (layer "F.Fab") hide)
+    (pad "1" smd roundrect (at -0.775 0) (size 0.9 0.95) (layers "F.Cu" "F.Paste" "F.Mask") (roundrect_rratio 0.25) (net 2 "VBUS_USB"))
+    (pad "2" smd roundrect (at 0.775 0) (size 0.9 0.95) (layers "F.Cu" "F.Paste" "F.Mask") (roundrect_rratio 0.25) (net 1 "GND"))
   )
   (footprint "Resistor_SMD:R_0603_1608Metric" (layer "F.Cu") (at 13.5 8.5)
@@
     (property "Reference" "Q_EPD" (at 0 -1.8) (layer "F.SilkS"))
     (property "Value" "SI1308EDL-T1-GE3" (at 0 1.8) (layer "F.Fab") hide)
-    (pad "1" smd roundrect (at -0.95 -0.65) (size 0.7 0.7) (layers "F.Cu" "F.Paste" "F.Mask") (roundrect_rratio 0.2) (net 24 "EPD_GDR"))
-    (pad "2" smd roundrect (at -0.95 0.65) (size 0.7 0.7) (layers "F.Cu" "F.Paste" "F.Mask") (roundrect_rratio 0.2) (net 25 "EPD_RESE"))
+    (pad "1" smd roundrect (at -0.95 -0.65) (size 0.7 0.7) (layers "F.Cu" "F.Paste" "F.Mask") (roundrect_rratio 0.2) (net 25 "EPD_RESE"))
+    (pad "2" smd roundrect (at -0.95 0.65) (size 0.7 0.7) (layers "F.Cu" "F.Paste" "F.Mask") (roundrect_rratio 0.2) (net 24 "EPD_GDR"))
     (pad "3" smd roundrect (at 0.95 0) (size 0.7 0.7) (layers "F.Cu" "F.Paste" "F.Mask") (roundrect_rratio 0.2) (net 54 "EPD_SW"))
   )
@@
   )
   (segment (start 58.225 20.25) (end 56.75 20.25) (width 0.20) (layer "F.Cu") (net 56))
-  (segment (start 33.55 34.35) (end 32.4 33.8) (width 0.20) (layer "F.Cu") (net 24))
+  (segment (start 33.55 35.65) (end 32.4 35.65) (width 0.20) (layer "F.Cu") (net 24))
+  (segment (start 32.4 35.65) (end 32.4 33.8) (width 0.20) (layer "F.Cu") (net 24))
+  (segment (start 33.55 34.35) (end 34.2 34.0) (width 0.20) (layer "F.Cu") (net 25))
+  (via (at 34.2 34.0) (size 0.60) (drill 0.30) (layers "F.Cu" "B.Cu") (net 25))
+  (segment (start 34.2 34.0) (end 34.2 37.4) (width 0.20) (layer "B.Cu") (net 25))
+  (segment (start 34.2 37.4) (end 30.0 37.4) (width 0.20) (layer "B.Cu") (net 25))
   (via (at 32.4 33.8) (size 0.60) (drill 0.30) (layers "F.Cu" "B.Cu") (net 24))
   (segment (start 32.4 33.8) (end 23.5 33.8) (width 0.20) (layer "B.Cu") (net 24))
@@
   (via (at 23.5 33.0) (size 0.60) (drill 0.30) (layers "F.Cu" "B.Cu") (net 6))
   (segment (start 23.5 33.0) (end 26.0 35.0) (width 0.35) (layer "In2.Cu") (net 6))
-  (segment (start 33.55 35.65) (end 33.55 37.4) (width 0.20) (layer "F.Cu") (net 25))
-  (segment (start 33.55 37.4) (end 30.0 37.4) (width 0.20) (layer "F.Cu") (net 25))
   (segment (start 39.25 17.71) (end 38.5 17.7) (width 0.20) (layer "F.Cu") (net 46))
   (via (at 38.5 17.7) (size 0.60) (drill 0.30) (layers "F.Cu" "B.Cu") (net 46))
@@
   (segment (start 61.50 6.00) (end 61.50 3.00) (width 0.20) (layer "F.Cu") (net 43))
   (segment (start 61.50 3.00) (end 62.00 2.15) (width 0.20) (layer "F.Cu") (net 43))
+  (segment (start 21.0 9.8) (end 22.8 12.8) (width 0.30) (layer "B.Cu") (net 2))
+  (via (at 22.8 12.8) (size 0.60) (drill 0.30) (layers "F.Cu" "B.Cu") (net 2))
+  (segment (start 22.8 12.8) (end 23.725 13.0) (width 0.30) (layer "F.Cu") (net 2))
+  (segment (start 25.275 13.0) (end 26.0 13.0) (width 0.30) (layer "F.Cu") (net 1))
+  (via (at 26.0 13.0) (size 0.60) (drill 0.30) (layers "F.Cu" "B.Cu") (net 1))
   (segment (start 21.0 9.8) (end 21.0 3.5) (width 0.50) (layer "In2.Cu") (net 2))
   (segment (start 21.0 3.5) (end 69.8 3.5) (width 0.50) (layer "In2.Cu") (net 2))

Commit message: fix(mainboard): clear DRC around charger bypass and EPD source route
Parts:
- moved C_IN 8.85 mm to (18.0, 7.00), turned to 180 degrees
Routing:
- net VBUS_USB: track 98.9 -> 96.6 mm
- net EPD_RESE: track 33.7 -> 34.9 mm
Changed lines of the file:
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@@
     (pad "2" smd roundrect (at 0.95 0) (size 1 1.45) (layers "F.Cu" "F.Paste" "F.Mask") (roundrect_rratio 0.25) (net 1 "GND"))
   )
-  (footprint "Capacitor_SMD:C_0603_1608Metric" (layer "F.Cu") (at 24.5 13.0)
+  (footprint "Capacitor_SMD:C_0603_1608Metric" (layer "F.Cu") (at 18.0 7.0 180)
     (property "Reference" "C_IN" (at 0 -1.4) (layer "F.SilkS"))
     (property "Value" "1uF/10V" (at 0 1.4) (layer "F.Fab") hide)
@@
   (segment (start 33.55 35.65) (end 32.4 35.65) (width 0.20) (layer "F.Cu") (net 24))
   (segment (start 32.4 35.65) (end 32.4 33.8) (width 0.20) (layer "F.Cu") (net 24))
-  (segment (start 33.55 34.35) (end 34.2 34.0) (width 0.20) (layer "F.Cu") (net 25))
-  (via (at 34.2 34.0) (size 0.60) (drill 0.30) (layers "F.Cu" "B.Cu") (net 25))
-  (segment (start 34.2 34.0) (end 34.2 37.4) (width 0.20) (layer "B.Cu") (net 25))
-  (segment (start 34.2 37.4) (end 30.0 37.4) (width 0.20) (layer "B.Cu") (net 25))
+  (segment (start 33.55 34.35) (end 34.8 34.0) (width 0.20) (layer "F.Cu") (net 25))
+  (via (at 34.8 34.0) (size 0.60) (drill 0.30) (layers "F.Cu" "B.Cu") (net 25))
+  (segment (start 34.8 34.0) (end 34.8 37.4) (width 0.20) (layer "B.Cu") (net 25))
+  (segment (start 34.8 37.4) (end 30.0 37.4) (width 0.20) (layer "B.Cu") (net 25))
   (via (at 32.4 33.8) (size 0.60) (drill 0.30) (layers "F.Cu" "B.Cu") (net 24))
   (segment (start 32.4 33.8) (end 23.5 33.8) (width 0.20) (layer "B.Cu") (net 24))
@@
   (segment (start 61.50 6.00) (end 61.50 3.00) (width 0.20) (layer "F.Cu") (net 43))
   (segment (start 61.50 3.00) (end 62.00 2.15) (width 0.20) (layer "F.Cu") (net 43))
-  (segment (start 21.0 9.8) (end 22.8 12.8) (width 0.30) (layer "B.Cu") (net 2))
-  (via (at 22.8 12.8) (size 0.60) (drill 0.30) (layers "F.Cu" "B.Cu") (net 2))
-  (segment (start 22.8 12.8) (end 23.725 13.0) (width 0.30) (layer "F.Cu") (net 2))
-  (segment (start 25.275 13.0) (end 26.0 13.0) (width 0.30) (layer "F.Cu") (net 1))
-  (via (at 26.0 13.0) (size 0.60) (drill 0.30) (layers "F.Cu" "B.Cu") (net 1))
+  (segment (start 21.0 7.0) (end 19.5 7.0) (width 0.30) (layer "In2.Cu") (net 2))
+  (via (at 19.5 7.0) (size 0.60) (drill 0.30) (layers "F.Cu" "B.Cu") (net 2))
+  (segment (start 19.5 7.0) (end 18.775 7.0) (width 0.30) (layer "F.Cu") (net 2))
+  (segment (start 17.225 7.0) (end 16.5 7.0) (width 0.30) (layer "F.Cu") (net 1))
+  (via (at 16.5 7.0) (size 0.60) (drill 0.30) (layers "F.Cu" "B.Cu") (net 1))
   (segment (start 21.0 9.8) (end 21.0 3.5) (width 0.50) (layer "In2.Cu") (net 2))
   (segment (start 21.0 3.5) (end 69.8 3.5) (width 0.50) (layer "In2.Cu") (net 2))

Commit message: fix(mainboard): move EPD source via clear of switch node
Routing:
- net EPD_RESE: track 34.9 -> 32.0 mm
Changed lines of the file:
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@@
   (segment (start 33.55 35.65) (end 32.4 35.65) (width 0.20) (layer "F.Cu") (net 24))
   (segment (start 32.4 35.65) (end 32.4 33.8) (width 0.20) (layer "F.Cu") (net 24))
-  (segment (start 33.55 34.35) (end 34.8 34.0) (width 0.20) (layer "F.Cu") (net 25))
-  (via (at 34.8 34.0) (size 0.60) (drill 0.30) (layers "F.Cu" "B.Cu") (net 25))
-  (segment (start 34.8 34.0) (end 34.8 37.4) (width 0.20) (layer "B.Cu") (net 25))
-  (segment (start 34.8 37.4) (end 30.0 37.4) (width 0.20) (layer "B.Cu") (net 25))
+  (segment (start 33.55 34.35) (end 32.5 34.35) (width 0.20) (layer "F.Cu") (net 25))
+  (via (at 32.5 34.35) (size 0.60) (drill 0.30) (layers "F.Cu" "B.Cu") (net 25))
+  (segment (start 32.5 34.35) (end 32.5 37.4) (width 0.20) (layer "B.Cu") (net 25))
+  (segment (start 32.5 37.4) (end 30.0 37.4) (width 0.20) (layer "B.Cu") (net 25))
   (via (at 32.4 33.8) (size 0.60) (drill 0.30) (layers "F.Cu" "B.Cu") (net 24))
   (segment (start 32.4 33.8) (end 23.5 33.8) (width 0.20) (layer "B.Cu") (net 24))

Commit message: fix(mainboard): extend charger safety timer for 3Ah battery
Parts:
- R_TMR: value 46.4k -> 68k
Changed lines of the file:
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@@
   (footprint "Resistor_SMD:R_0603_1608Metric" (layer "F.Cu") (at 21 8.5)
     (property "Reference" "R_TMR" (at 0 -1.4) (layer "F.SilkS"))
-    (property "Value" "46.4k" (at 0 1.4) (layer "F.Fab") hide)
+    (property "Value" "68k" (at 0 1.4) (layer "F.Fab") hide)
     (pad "1" smd roundrect (at -0.775 0) (size 0.9 0.95) (layers "F.Cu" "F.Paste" "F.Mask") (roundrect_rratio 0.25) (net 62 "CHG_TMR"))
     (pad "2" smd roundrect (at 0.775 0) (size 0.9 0.95) (layers "F.Cu" "F.Paste" "F.Mask") (roundrect_rratio 0.25) (net 1 "GND"))

Commit message: fix(mainboard): separate EPD gate and source routing
Routing:
- net EPD_RESE: track 32.0 -> 33.4 mm
Changed lines of the file:
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@@
   (segment (start 33.55 35.65) (end 32.4 35.65) (width 0.20) (layer "F.Cu") (net 24))
   (segment (start 32.4 35.65) (end 32.4 33.8) (width 0.20) (layer "F.Cu") (net 24))
-  (segment (start 33.55 34.35) (end 32.5 34.35) (width 0.20) (layer "F.Cu") (net 25))
-  (via (at 32.5 34.35) (size 0.60) (drill 0.30) (layers "F.Cu" "B.Cu") (net 25))
-  (segment (start 32.5 34.35) (end 32.5 37.4) (width 0.20) (layer "B.Cu") (net 25))
-  (segment (start 32.5 37.4) (end 30.0 37.4) (width 0.20) (layer "B.Cu") (net 25))
+  (segment (start 33.55 34.35) (end 34.25 34.35) (width 0.20) (layer "F.Cu") (net 25))
+  (via (at 34.25 34.35) (size 0.60) (drill 0.30) (layers "F.Cu" "B.Cu") (net 25))
+  (segment (start 34.25 34.35) (end 34.25 37.4) (width 0.20) (layer "B.Cu") (net 25))
+  (segment (start 34.25 37.4) (end 30.0 37.4) (width 0.20) (layer "B.Cu") (net 25))
   (via (at 32.4 33.8) (size 0.60) (drill 0.30) (layers "F.Cu" "B.Cu") (net 24))
   (segment (start 32.4 33.8) (end 23.5 33.8) (width 0.20) (layer "B.Cu") (net 24))

Commit message: fix(mainboard): move EPD pump inner-layer route clear of source via
Routing:
- net EPD_PUMP: track 21.6 -> 16.6 mm
Changed lines of the file:
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@@
   (segment (start 40.05 36.5) (end 39.0 36.4) (width 0.24) (layer "F.Cu") (net 55))
   (via (at 39.0 36.4) (size 0.60) (drill 0.30) (layers "F.Cu" "B.Cu") (net 55))
-  (segment (start 39.0 36.4) (end 34.0 36.4) (width 0.24) (layer "In2.Cu") (net 55))
-  (segment (start 34.0 36.4) (end 34.0 31.6) (width 0.24) (layer "In2.Cu") (net 55))
-  (segment (start 34.0 31.6) (end 42.7 31.6) (width 0.24) (layer "In2.Cu") (net 55))
+  (segment (start 39.0 36.4) (end 36.5 36.4) (width 0.24) (layer "In2.Cu") (net 55))
+  (segment (start 36.5 36.4) (end 36.5 31.6) (width 0.24) (layer "In2.Cu") (net 55))
+  (segment (start 36.5 31.6) (end 42.7 31.6) (width 0.24) (layer "In2.Cu") (net 55))
   (segment (start 42.7 31.6) (end 42.7 32.4) (width 0.24) (layer "In2.Cu") (net 55))
   (via (at 42.7 32.4) (size 0.60) (drill 0.30) (layers "F.Cu" "B.Cu") (net 55))

Commit message: fix(mainboard): orient USB-C to board edge and reroute port nets
Parts:
- moved J1 9.00 mm to (76.0, 0.00), turned to 180 degrees
Routing:
- net USB_CC2: track 38.0 -> 6.75 mm
- net USB_CC1: track 10.8 -> 2.60 mm, vias 2 -> 0
- net USB_D-_CONN: track 16.0 -> 8.67 mm, vias 2 -> 0
- net VBUS_USB: track 96.6 -> 90.6 mm
- net USB_D+_CONN: track 12.0 -> 13.0 mm
Changed lines of the file:
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@@
     (property "Reference" "H4" (at 0 -2.5) (layer "F.SilkS") hide)
     (pad "" np_thru_hole circle (at 0 0) (size 2.7 2.7) (drill 2.7) (layers "*.Cu" "*.Mask")))
-  (footprint "ENKU_Clock:HRO-TYPE-C-31-M-12" (layer "F.Cu") (at 76 9)
+  (footprint "ENKU_Clock:HRO-TYPE-C-31-M-12" (layer "F.Cu") (at 76 0 180)
     (property "Reference" "J1" (at 0 1.8) (layer "F.SilkS"))
     (property "Value" "USB-C" (at 0 1.15) (layer "F.Fab") hide)
@@
   (segment (start 39.25 17.71) (end 38.5 17.7) (width 0.20) (layer "F.Cu") (net 46))
   (via (at 38.5 17.7) (size 0.60) (drill 0.30) (layers "F.Cu" "B.Cu") (net 46))
-  (segment (start 73.55 2.03) (end 73.55 1.85) (width 0.25) (layer "F.Cu") (net 2))
-  (via (at 73.55 1.85) (size 0.50) (drill 0.30) (layers "F.Cu" "B.Cu") (net 2))
-  (segment (start 73.55 1.85) (end 74.2 1.85) (width 0.30) (layer "In2.Cu") (net 2))
-  (segment (start 74.2 1.85) (end 74.2 4.6) (width 0.35) (layer "In2.Cu") (net 2))
-  (segment (start 74.2 4.6) (end 69.8 4.6) (width 0.35) (layer "In2.Cu") (net 2))
-  (segment (start 78.45 2.03) (end 78.45 1.85) (width 0.25) (layer "F.Cu") (net 2))
-  (via (at 78.45 1.85) (size 0.50) (drill 0.30) (layers "F.Cu" "B.Cu") (net 2))
-  (segment (start 78.45 1.85) (end 77.8 1.85) (width 0.30) (layer "In2.Cu") (net 2))
-  (segment (start 77.8 1.85) (end 77.8 4.6) (width 0.35) (layer "In2.Cu") (net 2))
-  (segment (start 77.8 4.6) (end 69.8 4.6) (width 0.35) (layer "In2.Cu") (net 2))
   (segment (start 73.425 31.25) (end 76.0 31.25) (width 0.20) (layer "F.Cu") (net 20))
   (via (at 76.0 31.25) (size 0.60) (drill 0.30) (layers "F.Cu" "B.Cu") (net 20))
@@
   (segment (start 24.5 20.5) (end 24.5 21.4) (width 0.20) (layer "B.Cu") (net 8))
   (segment (start 55.0 21.4) (end 55.0 21.0) (width 0.20) (layer "B.Cu") (net 8))
-  (segment (start 79.725 15.2) (end 79.725 10.5) (width 0.20) (layer "F.Cu") (net 22))
   (segment (start 81.275 10.5) (end 81.275 11.5) (width 0.20) (layer "F.Cu") (net 1))
   (via (at 81.275 11.5) (size 0.60) (drill 0.30) (layers "F.Cu" "B.Cu") (net 1))
@@
   (via (at 53.7 26.2) (size 0.60) (drill 0.30) (layers "F.Cu" "B.Cu") (net 9))
   (segment (start 53.7 26.2) (end 53.7 26.0) (width 0.20) (layer "B.Cu") (net 9))
-  (segment (start 82.8 15.2) (end 79.725 15.2) (width 0.20) (layer "F.Cu") (net 22))
     (via (at 21.0 9.8) (size 0.7) (drill 0.3) (layers "F.Cu" "B.Cu") (net 2))
     (segment (start 21.0 9.8) (end 20.75 10.5375) (width 0.3) (layer "F.Cu") (net 2))
@@
   (via (at 73.0 40.8) (size 0.60) (drill 0.30) (layers "F.Cu" "B.Cu") (net 42))
   (segment (start 73.0 40.8) (end 73.0 42.0) (width 0.30) (layer "F.Cu") (net 42))
-  (segment (start 75.75 2.03) (end 75.75 2.40) (width 0.20) (layer "F.Cu") (net 59))
-  (via (at 75.75 2.40) (size 0.50) (drill 0.20) (layers "F.Cu" "B.Cu") (net 59))
-  (segment (start 76.75 2.03) (end 76.75 2.40) (width 0.20) (layer "F.Cu") (net 59))
-  (via (at 76.75 2.40) (size 0.50) (drill 0.20) (layers "F.Cu" "B.Cu") (net 59))
-  (segment (start 75.75 2.40) (end 74.0 2.40) (width 0.20) (layer "B.Cu") (net 59))
-  (segment (start 76.75 2.40) (end 74.0 2.40) (width 0.20) (layer "B.Cu") (net 59))
-  (segment (start 74.0 2.40) (end 74.0 3.70) (width 0.20) (layer "B.Cu") (net 59))
-  (segment (start 74.0 3.70) (end 70.8 3.70) (width 0.20) (layer "B.Cu") (net 59))
-  (via (at 70.8 3.70) (size 0.60) (drill 0.30) (layers "F.Cu" "B.Cu") (net 59))
-  (segment (start 70.8 3.70) (end 69.0 5.05) (width 0.20) (layer "F.Cu") (net 59))
-  (segment (start 75.25 2.03) (end 75.25 3.60) (width 0.20) (layer "F.Cu") (net 60))
-  (segment (start 76.25 2.03) (end 76.25 3.60) (width 0.20) (layer "F.Cu") (net 60))
-  (segment (start 75.25 3.60) (end 76.25 3.60) (width 0.20) (layer "F.Cu") (net 60))
-  (segment (start 76.25 3.60) (end 76.25 5.40) (width 0.20) (layer "F.Cu") (net 60))
-  (via (at 76.25 5.40) (size 0.60) (drill 0.30) (layers "F.Cu" "B.Cu") (net 60))
-  (segment (start 76.25 5.40) (end 76.25 8.00) (width 0.20) (layer "B.Cu") (net 60))
-  (segment (start 76.25 8.00) (end 71.00 8.00) (width 0.20) (layer "B.Cu") (net 60))
-  (via (at 71.00 8.00) (size 0.60) (drill 0.30) (layers "F.Cu" "B.Cu") (net 60))
-  (segment (start 71.00 8.00) (end 69.0 6.95) (width 0.20) (layer "F.Cu") (net 60))
+  (segment (start 77.25 7.695) (end 79.725 8.50) (width 0.20) (layer "F.Cu") (net 21))
+  (segment (start 74.25 7.695) (end 74.25 8.60) (width 0.20) (layer "F.Cu") (net 22))
+  (via (at 74.25 8.60) (size 0.60) (drill 0.30) (layers "F.Cu" "B.Cu") (net 22))
+  (segment (start 74.25 8.60) (end 78.90 10.50) (width 0.20) (layer "B.Cu") (net 22))
+  (via (at 78.90 10.50) (size 0.60) (drill 0.30) (layers "F.Cu" "B.Cu") (net 22))
+  (segment (start 78.90 10.50) (end 79.725 10.50) (width 0.20) (layer "F.Cu") (net 22))
+  (segment (start 76.25 7.695) (end 76.25 8.15) (width 0.20) (layer "F.Cu") (net 59))
+  (via (at 76.25 8.15) (size 0.50) (drill 0.20) (layers "F.Cu" "B.Cu") (net 59))
+  (segment (start 75.25 7.695) (end 75.25 8.15) (width 0.20) (layer "F.Cu") (net 59))
+  (via (at 75.25 8.15) (size 0.50) (drill 0.20) (layers "F.Cu" "B.Cu") (net 59))
+  (segment (start 76.25 8.15) (end 72.00 8.15) (width 0.20) (layer "B.Cu") (net 59))
+  (segment (start 75.25 8.15) (end 72.00 8.15) (width 0.20) (layer "B.Cu") (net 59))
+  (segment (start 72.00 8.15) (end 70.50 5.50) (width 0.20) (layer "B.Cu") (net 59))
+  (via (at 70.50 5.50) (size 0.60) (drill 0.30) (layers "F.Cu" "B.Cu") (net 59))
+  (segment (start 70.50 5.50) (end 69.0 5.05) (width 0.20) (layer "F.Cu") (net 59))
+  (segment (start 75.75 7.695) (end 76.25 7.20) (width 0.20) (layer "F.Cu") (net 60))
+  (segment (start 76.75 7.695) (end 76.25 7.20) (width 0.20) (layer "F.Cu") (net 60))
+  (segment (start 76.25 7.20) (end 71.00 7.20) (width 0.20) (layer "F.Cu") (net 60))
+  (segment (start 71.00 7.20) (end 69.0 6.95) (width 0.20) (layer "F.Cu") (net 60))
+  (segment (start 73.55 7.695) (end 73.55 9.10) (width 0.35) (layer "F.Cu") (net 2))
+  (via (at 73.55 9.10) (size 0.70) (drill 0.30) (layers "F.Cu" "B.Cu") (net 2))
+  (segment (start 78.45 7.695) (end 78.45 9.10) (width 0.35) (layer "F.Cu") (net 2))
+  (via (at 78.45 9.10) (size 0.70) (drill 0.30) (layers "F.Cu" "B.Cu") (net 2))
+  (segment (start 73.55 9.10) (end 69.80 4.60) (width 0.50) (layer "In2.Cu") (net 2))
+  (segment (start 78.45 9.10) (end 73.55 9.10) (width 0.50) (layer "In2.Cu") (net 2))
   (segment (start 69.0 6.0) (end 70.20 5.80) (width 0.35) (layer "F.Cu") (net 2))
   (via (at 70.20 5.80) (size 0.70) (drill 0.30) (layers "F.Cu" "B.Cu") (net 2))
@@
   (segment (start 43.275 38.5) (end 42.70 39.50) (width 0.20) (layer "F.Cu") (net 35))
   (via (at 42.70 39.50) (size 0.60) (drill 0.30) (layers "F.Cu" "B.Cu") (net 35))
-  (via (at 78.80 7.00) (size 0.60) (drill 0.30) (layers "F.Cu" "B.Cu") (net 21))
-  (segment (start 78.80 7.00) (end 79.725 8.50) (width 0.20) (layer "F.Cu") (net 21))
   (segment (start 46.275 38.5) (end 47.75 40.30) (width 0.20) (layer "F.Cu") (net 36))
   (segment (start 46.25 41.625) (end 46.25 40.20) (width 0.22) (layer "F.Cu") (net 1))
@@
   (segment (start 56.75 3.74) (end 58.00 2.50) (width 0.22) (layer "F.Cu") (net 1))
   (via (at 58.00 2.50) (size 0.60) (drill 0.30) (layers "F.Cu" "B.Cu") (net 1))
-  (segment (start 74.75 2.03) (end 74.75 7.00) (width 0.20) (layer "F.Cu") (net 21))
-  (via (at 74.75 7.00) (size 0.60) (drill 0.30) (layers "F.Cu" "B.Cu") (net 21))
-  (segment (start 74.75 7.00) (end 78.80 7.00) (width 0.20) (layer "In1.Cu") (net 21))
   (segment (start 34.0 21.5) (end 35.0 28.0) (width 0.20) (layer "In2.Cu") (net 47))
   (via (at 35.0 28.0) (size 0.60) (drill 0.30) (layers "F.Cu" "B.Cu") (net 47))
@@
   (via (at 40.00 22.80) (size 0.60) (drill 0.30) (layers "F.Cu" "B.Cu") (net 47))
   (segment (start 40.00 22.80) (end 36.0 21.0) (width 0.20) (layer "In2.Cu") (net 47))
-  (via (at 86.50 14.00) (size 0.60) (drill 0.30) (layers "F.Cu" "B.Cu") (net 22))
-  (segment (start 86.50 14.00) (end 81.00 14.00) (width 0.20) (layer "F.Cu") (net 22))
-  (segment (start 81.00 14.00) (end 79.725 10.50) (width 0.20) (layer "F.Cu") (net 22))
   (segment (start 23.45 24.80) (end 21.50 32.50) (width 0.20) (layer "In2.Cu") (net 64))
   (via (at 21.50 32.50) (size 0.60) (drill 0.30) (layers "F.Cu" "B.Cu") (net 64))
@@
   (segment (start 44.0 10.0) (end 44.0 16.5) (width 0.20) (layer "In1.Cu") (net 44))
   (segment (start 44.0 16.5) (end 57.0 16.5) (width 0.20) (layer "In1.Cu") (net 44))
-  (via (at 86.80 7.00) (size 0.60) (drill 0.30) (layers "F.Cu" "B.Cu") (net 22))
-  (segment (start 86.80 7.00) (end 86.80 14.00) (width 0.20) (layer "B.Cu") (net 22))
   (segment (start 56.75 5.01) (end 54.50 6.00) (width 0.20) (layer "F.Cu") (net 50))
   (via (at 54.50 6.00) (size 0.60) (drill 0.30) (layers "F.Cu" "B.Cu") (net 50))
@@
   (segment (start 45.50 44.00) (end 45.50 41.50) (width 0.20) (layer "In2.Cu") (net 33))
   (segment (start 45.50 41.50) (end 46.00 41.00) (width 0.20) (layer "In2.Cu") (net 33))
-  (segment (start 81.50 6.00) (end 86.80 6.00) (width 0.20) (layer "F.Cu") (net 22))
-  (segment (start 86.80 6.00) (end 86.80 7.00) (width 0.20) (layer "F.Cu") (net 22))
-  (segment (start 77.75 2.03) (end 77.75 4.20) (width 0.20) (layer "F.Cu") (net 22))
-  (segment (start 77.75 4.20) (end 81.50 4.20) (width 0.20) (layer "F.Cu") (net 22))
-  (segment (start 81.50 4.20) (end 81.50 6.00) (width 0.20) (layer "F.Cu") (net 22))
   (segment (start 45.25 41.625) (end 45.25 40.40) (width 0.20) (layer "F.Cu") (net 6))
   (segment (start 45.75 41.625) (end 45.75 40.40) (width 0.20) (layer "F.Cu") (net 6))
