File: hardware/daughterboards/wake-led/wake-led-board-reva.kicad_pcb (KiCad board)
At the start: 2 copper layers, 78 x 8 mm, 13 parts, among them J1 SM02B-GHS-TB

Commit message: fix(hardware): remove audio via-in-pad and correct wake LED polarity marks
Changed lines of the file:
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@@
   (gr_rect (start 0 0) (end 78 8)
     (stroke (width 0.05) (type default)) (fill none) (layer "Edge.Cuts"))
-  (gr_circle (center 34 6.49) (end 34.55 6.49)
-    (stroke (width 0) (type solid)) (fill solid) (layer "B.Mask"))
   (gr_text "ENKU CLOCK WAKE LIGHT REV A"
     (at 39 4.0) (layer "B.SilkS")
@@
     (property "Value" "NFSW757G-V3 2700K" (at 0 2.1) (layer "F.Fab") hide)
     (fp_rect (start -1.5 -1.5) (end 1.5 1.5) (stroke (width 0.08) (type default)) (fill none) (layer "F.Fab"))
-    (fp_line (start -2.0 -0.4) (end -2.0 0.4) (stroke (width 0.15) (type default)) (layer "F.SilkS"))
+    (fp_line (start -0.5 2.35) (end 0.5 2.35) (stroke (width 0.15) (type default)) (layer "F.SilkS"))
     (pad "2" smd rect (at 0 -1.1) (size 2.3 0.58) (layers "F.Cu" "F.Paste" "F.Mask") (net 2 "LED1_A"))
     (pad "2" smd rect (at 0 -1.68) (size 3.15 0.7) (layers "F.Cu" "F.Paste" "F.Mask") (net 2 "LED1_A"))
@@
     (property "Value" "NFSW757G-V3 2700K" (at 0 2.1) (layer "F.Fab") hide)
     (fp_rect (start -1.5 -1.5) (end 1.5 1.5) (stroke (width 0.08) (type default)) (fill none) (layer "F.Fab"))
-    (fp_line (start -2.0 -0.4) (end -2.0 0.4) (stroke (width 0.15) (type default)) (layer "F.SilkS"))
+    (fp_line (start -0.5 2.35) (end 0.5 2.35) (stroke (width 0.15) (type default)) (layer "F.SilkS"))
     (pad "2" smd rect (at 0 -1.1) (size 2.3 0.58) (layers "F.Cu" "F.Paste" "F.Mask") (net 3 "LED2_A"))
     (pad "2" smd rect (at 0 -1.68) (size 3.15 0.7) (layers "F.Cu" "F.Paste" "F.Mask") (net 3 "LED2_A"))
@@
     (property "Value" "NFSW757G-V3 2700K" (at 0 2.1) (layer "F.Fab") hide)
     (fp_rect (start -1.5 -1.5) (end 1.5 1.5) (stroke (width 0.08) (type default)) (fill none) (layer "F.Fab"))
-    (fp_line (start -2.0 -0.4) (end -2.0 0.4) (stroke (width 0.15) (type default)) (layer "F.SilkS"))
+    (fp_line (start -0.5 2.35) (end 0.5 2.35) (stroke (width 0.15) (type default)) (layer "F.SilkS"))
     (pad "2" smd rect (at 0 -1.1) (size 2.3 0.58) (layers "F.Cu" "F.Paste" "F.Mask") (net 4 "LED3_A"))
     (pad "2" smd rect (at 0 -1.68) (size 3.15 0.7) (layers "F.Cu" "F.Paste" "F.Mask") (net 4 "LED3_A"))
@@
     (property "Value" "NFSW757G-V3 2700K" (at 0 2.1) (layer "F.Fab") hide)
     (fp_rect (start -1.5 -1.5) (end 1.5 1.5) (stroke (width 0.08) (type default)) (fill none) (layer "F.Fab"))
-    (fp_line (start -2.0 -0.4) (end -2.0 0.4) (stroke (width 0.15) (type default)) (layer "F.SilkS"))
+    (fp_line (start -0.5 2.35) (end 0.5 2.35) (stroke (width 0.15) (type default)) (layer "F.SilkS"))
     (pad "2" smd rect (at 0 -1.1) (size 2.3 0.58) (layers "F.Cu" "F.Paste" "F.Mask") (net 5 "LED4_A"))
     (pad "2" smd rect (at 0 -1.68) (size 3.15 0.7) (layers "F.Cu" "F.Paste" "F.Mask") (net 5 "LED4_A"))
@@
     (property "Value" "NFSW757G-V3 2700K" (at 0 2.1) (layer "F.Fab") hide)
     (fp_rect (start -1.5 -1.5) (end 1.5 1.5) (stroke (width 0.08) (type default)) (fill none) (layer "F.Fab"))
-    (fp_line (start -2.0 -0.4) (end -2.0 0.4) (stroke (width 0.15) (type default)) (layer "F.SilkS"))
+    (fp_line (start -0.5 2.35) (end 0.5 2.35) (stroke (width 0.15) (type default)) (layer "F.SilkS"))
     (pad "2" smd rect (at 0 -1.1) (size 2.3 0.58) (layers "F.Cu" "F.Paste" "F.Mask") (net 6 "LED5_A"))
     (pad "2" smd rect (at 0 -1.68) (size 3.15 0.7) (layers "F.Cu" "F.Paste" "F.Mask") (net 6 "LED5_A"))
@@
     (property "Value" "NFSW757G-V3 2700K" (at 0 2.1) (layer "F.Fab") hide)
     (fp_rect (start -1.5 -1.5) (end 1.5 1.5) (stroke (width 0.08) (type default)) (fill none) (layer "F.Fab"))
-    (fp_line (start -2.0 -0.4) (end -2.0 0.4) (stroke (width 0.15) (type default)) (layer "F.SilkS"))
+    (fp_line (start -0.5 2.35) (end 0.5 2.35) (stroke (width 0.15) (type default)) (layer "F.SilkS"))
     (pad "2" smd rect (at 0 -1.1) (size 2.3 0.58) (layers "F.Cu" "F.Paste" "F.Mask") (net 7 "LED6_A"))
     (pad "2" smd rect (at 0 -1.68) (size 3.15 0.7) (layers "F.Cu" "F.Paste" "F.Mask") (net 7 "LED6_A"))
